Commit message: agregué las graficas de fuerza la caminata con trayectoria sinusoidal

File: solo12-pybullet/Models/wedge.urdf (robot description, URDF)
Before this commit: robot obstacle, 1 links, 0 joints
Links:
- link base_link: geometry collision mesh filename=/home/renzo/Documents/RLE/Codigos/rle_127/solo12-pybullet/M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 scale=0.5; visual mesh filename=//home/renzo/Documents/RLE/Codigos/rle_127/solo12-pybullet/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 scale=0.5
